File: kicad/6502/v1/6502_adapter.sch (KiCad schematic (older format))
At the start: 53 parts, among them P1 Conn_02x20_Odd_Even, P2 Conn_02x20_Odd_Even, P3 Conn_01x03, SW1 SW_Push, SW2 SW_Push, U1 WD65C02, U2 74LVC4245, U3 74LVC4245, U4 74LVC4245, U5 74LVC4245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

Commit message: kicad 6502: added weak pullups to 6502 control signals
Change-Id: Iba7afce3f12305b795a8ec8d95fa880e29d4dc03
Parts:
- added R16, R17, R18, R19, R20: 22K, Resistor_SMD:R_0805_2012Metric_Pad1.15x1.40mm_HandSolder, symbol Device:R_Small
- D4, D5: value MBR130 -> PMEG3010BEA; footprint Diode_SMD:D_0805_2012Metric_Pad1.15x1.40mm_HandSolder -> Diode_SMD:D_SOD-323_HandSoldering
Connections:
- wire segments 206 -> 226
Other:
- moved on the sheet: C15, R14
